File: QuadQuantizer/QuadQuantizer.kicad_pcb (KiCad board)
At the start: 2 copper layers, 76.8 x 73.7 mm, 71 parts, among them J1 OLED, J2 R_ENC, J3 CV_IN, J4 CV_OUT, J5 TR_OUT, J6 POWER, M1 RP2040zero, U1 24LC04, U2 MAX5715BAUD, U3 TL074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

Commit message: Add files via upload
Other:
- board text removed: "JLCJLCJLCJLC"
